File: Touch Switch.kicad_sch (KiCad schematic)
At the start: 25 parts, among them J1 Conn_01x03_Pin, T1 Transformer_1P_2S, U1 SCJT1117B-3.3-A

Commit message: Schematic finished
Parts:
- removed D1: KBPC1501W, Diode_THT:Diode_Bridge_GeneSiC_KBPC_W, symbol Diode_Bridge:KBPC1501W
- removed R4: R1,5, symbol Device:R
- added C7: 100nF, symbol Device:C
- added C8: C, symbol Device:C
- added D1: D_Bridge_+-AA, Diode_SMD:Diode_Bridge_Diotec_ABS, symbol Device:D_Bridge_+-AA
- added D5, D6, D7, D8: D, Diode_SMD:D_SOD-123, symbol Device:D
- added F1: 68R, footprint:fuse, symbol Device:Fuse
- added J2: Conn_02x04_Counter_Clockwise, Diode_SMD:D_SMA, symbol Connector_Generic:Conn_02x04_Counter_Clockwise
- added K1, K2, K3, K4: Relay_SPST-NO, footprint:relay, symbol Relay:Relay_SPST-NO
- added Q1, Q2, Q3, Q5: MMBT3904, Package_TO_SOT_SMD:SOT-23, symbol Transistor_BJT:MMBT3904
- added R11, R12, R13, R14: 10K, Resistor_SMD:R_1206_3216Metric, symbol Device:R
- added R15: 100, symbol Device:R
- added R16: 1,5R, Resistor_SMD:R_1206_3216Metric, symbol Device:R
- C4: value C -> 100nF
- C6: value C_Polarized -> 4,7µF; footprint (none) -> Capacitor_SMD:C_0805_2012Metric
- D2, D3, D4, J1: footprint (none) -> Diode_SMD:D_SMA
- L1: value L_Ferrite -> 3.0mH; footprint (none) -> Inductor_THT:L_Radial_D7.5mm_P3.50mm_Fastron_07P
- R1: value R -> 5,6K
- R10, R5, R6, R9: footprint (none) -> Resistor_SMD:R_1206_3216Metric
- R2: value R -> 1K; footprint (none) -> Resistor_SMD:R_1206_3216Metric
- R8: value R -> 100
- S7133S1: renamed from S7133S; footprint (none) -> Package_SO:SOP-8_3.9x4.9mm_P1.27mm
Connections:
- net +3.3V: now also J2.8 (Pin_8)
- net +5V: now also D5.1 (K), D6.1 (K), D7.1 (K), D8.1 (K), K1.A1, K2.A1, K3.A1, K4.A1
- net GND: now also C8.2, D1.2 (-), R16.2
- net GND2: now also J2.7 (Pin_7), Q1.2 (E), Q2.2 (E), Q3.2 (E), Q5.2 (E), R11.2, R12.2, R13.2, R14.2
- net L: now also F1.1, K1.13, K2.13, K3.13, K4.13
- net N: now also C7.2, D1.4
- net at L1.1, R1.2: now also C8.1, D1.1 (+)
- net at S7133S1.4 (CS): now also R16.1
- net at C5.2, R3.2, R7.2: now also R15.1; no longer D3.1 (K)
- new net: D7.2 (A), K4.A2, Q3.3 (C)
- new net: D5.2 (A), K1.A2, Q5.3 (C)
- new net: D6.2 (A), K2.A2, Q1.3 (C)
- new net: D3.1 (K), R15.2
- new net: D8.2 (A), K3.A2, Q2.3 (C)
- new net: C7.1, D1.3, F1.2
- new net CT1: J2.5 (Pin_5), Q5.1 (B), R11.1
- new net CT2: J2.4 (Pin_4), Q3.1 (B), R14.1
- new net CT3: J2.3 (Pin_3), Q1.1 (B), R12.1
- new net CT4: J2.2 (Pin_2), Q2.1 (B), R13.1
- new net R1: K1.14
- new net R2: K4.14
- new net R3: K2.14
- new net R4: K3.14
Other:
- moved on the sheet: C1, C5, C6, D3, D4, L1, R1, R10, R3, R5, R6, R7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

Commit message: PCB started
Parts:
- removed C8: C, symbol Device:C
- added J3, J4, J5, J6: Conn_01x01_Pin, symbol Connector:Conn_01x01_Pin
- C1: value 2,2µF -> 2,2µF - 400V; footprint (none) -> footprint:PFR5101J400J11L4BULK
- C2: value 470µF -> 470µF - 10V; footprint (none) -> Capacitor_THT:CP_Radial_D6.3mm_P2.50mm
- C3: value 330µF -> 330µF - 10V; footprint (none) -> Capacitor_THT:CP_Radial_D6.3mm_P2.50mm
- C4: value 100nF -> 100nF - 10V; footprint (none) -> Capacitor_SMD:C_0805_2012Metric
- C5: value 100pF -> 100pF - 400V; footprint (none) -> footprint:B32524R6225J000
- C6: value 4,7µF -> 4,7µF - 25V
- C7: value 100nF -> 100nF - 400V; footprint (none) -> footprint:MKP-X2-100NR10310
- J1: footprint Diode_SMD:D_SMA -> (none)
- J2: footprint Diode_SMD:D_SMA -> Connector_PinSocket_2.54mm:PinSocket_2x04_P2.54mm_Vertical
- R1, R8: footprint (none) -> Resistor_SMD:R_0805_2012Metric
- R11, R12, R13, R14: footprint Resistor_SMD:R_1206_3216Metric -> Resistor_SMD:R_0805_2012Metric
- R15, R3, R7: footprint (none) -> Resistor_SMD:R_1206_3216Metric
Connections:
- net R1: now also J3.1 (Pin_1)
- net R2: now also J4.1 (Pin_1)
- net R3: now also J5.1 (Pin_1)
- net R4: now also J6.1 (Pin_1)
Other:
- moved on the sheet: C5, C6, D3, D4, J2, R10, R15, R16, R3, R5, R6, R7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

Commit message: PCB V1
Parts:
- removed S7133S1: ~, Package_SO:SOP-8_3.9x4.9mm_P1.27mm, symbol Library:S7133S
- added S713XS1: ~, Package_SO:SOP-8_3.9x4.9mm_P1.27mm, symbol Library:S7133S
- C1: footprint footprint:PFR5101J400J11L4BULK -> Capacitor_THT:CP_Radial_D8.0mm_P3.50mm
- C5: footprint footprint:B32524R6225J000 -> footprint:PFR5101J400J11L4BULK
- J1: footprint (none) -> Connector_PinHeader_2.54mm:PinHeader_1x03_P2.54mm_Vertical
- J3, J4, J5, J6: footprint (none) -> Connector_PinHeader_2.54mm:PinHeader_1x01_P2.54mm_Vertical
- T1: footprint (none) -> footprint:transformer
Connections:
- net CT1: now also Q3.1 (B), R14.1; no longer Q5.1 (B), R11.1
- net CT2: now also Q5.1 (B), R11.1; no longer Q3.1 (B), R14.1
- net CT3: now also Q2.1 (B), R13.1; no longer Q1.1 (B), R12.1
- net CT4: now also Q1.1 (B), R12.1; no longer Q2.1 (B), R13.1
- net GND: now also S713XS1.8 (GND)
- net L: no longer F1.1, J1.1 (Pin_1)
- net Prim: now also S713XS1.5 (C), S713XS1.6 (C)
- net VCC_IC: now also S713XS1.1 (VCC)
- net at R5.1, R6.2: now also S713XS1.2 (FB)
- net at R16.1: now also S713XS1.4 (CS)
- new net L1: F1.1, J1.1 (Pin_1)
Changed lines of the file:
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@@
 	(wire
 		(pts
-			(xy 180.34 100.33) (xy 180.34 97.79)
+			(xy 176.53 97.79) (xy 176.53 99.06)
 		)
 		(stroke
@@
 		)
 	)
-	(global_label "CT3"
-		(shape input)
-		(at 29.21 152.4 180)
-		(fields_autoplaced yes)
-		(effects
-			(font
-				(size 1.27 1.27)
-			)
-			(justify right)
-		)
-		(property "Intersheetrefs" "${INTERSHEET_REFS}"
-			(at 22.7777 152.4 0)
-			(effects
-				(font
-					(size 1.27 1.27)
-				)
-				(justify right)
-				(hide yes)
-			)
-		)
-	)
 	(global_label "Aux"
 		(shape input)
@@
 		)
 	)
-	(global_label "L"
+	(global_label "L1"
 		(shape input)
 		(at 30.48 21.59 180)
@@
 		)
 		(property "Intersheetrefs" "${INTERSHEET_REFS}"
-			(at 26.4667 21.59 0)
+			(at 25.2572 21.59 0)
 			(effects
 				(font
@@
 		)
 	)
-	(global_label "CT1"
+	(global_label "CT2"
 		(shape input)
 		(at 29.21 97.79 180)
@@
 		)
 	)
+	(global_label "CT1"
+		(shape input)
+		(at 88.9 96.52 180)
+		(fields_autoplaced yes)
+		(effects
+			(font
+				(size 1.27 1.27)
+			)
+			(justify right)
+		)
+		(property "Intersheetrefs" "${INTERSHEET_REFS}"
+			(at 82.4677 96.52 0)
+			(effects
+				(font
+					(size 1.27 1.27)
+				)
+				(justify right)
+				(hide yes)
+			)
+		)
+	)
 	(global_label "Prim"
 		(shape input)
@@
 		)
 	)
-	(global_label "CT4"
+	(global_label "CT3"
 		(shape input)
 		(at 85.09 152.4 180)
@@
 		)
 	)
-	(global_label "CT2"
+	(global_label "L"
 		(shape input)
-		(at 88.9 96.52 180)
+		(at 116.84 144.78 270)
 		(fields_autoplaced yes)
 		(effects
@@
 		)
 		(property "Intersheetrefs" "${INTERSHEET_REFS}"
-			(at 82.4677 96.52 0)
+			(at 116.84 148.7933 90)
 			(effects
 				(font
@@
 		)
 	)
-	(global_label "L"
+	(global_label "CT4"
 		(shape input)
-		(at 116.84 144.78 270)
+		(at 29.21 152.4 180)
 		(fields_autoplaced yes)
 		(effects
@@
 		)
 		(property "Intersheetrefs" "${INTERSHEET_REFS}"
-			(at 116.84 148.7933 90)
+			(at 22.7777 152.4 0)
 			(effects
 				(font
@@
 			)
 		)
-		(property "Footprint" "footprint:PFR5101J400J11L4BULK"
+		(property "Footprint" "Capacitor_THT:CP_Radial_D8.0mm_P3.50mm"
 			(at 84.7852 39.37 0)
 			(effects
@@
 	)
 	(symbol
-		(lib_id "Library:S7133S")
-		(at 180.34 83.82 0)
-		(unit 1)
-		(exclude_from_sim no)
-		(in_bom yes)
-		(on_board yes)
-		(dnp no)
-		(property "Reference" "S7133S1"
-			(at 167.386 97.028 0)
-			(effects
-				(font
-					(size 1.27 1.27)
-				)
-				(justify left)
-			)
-		)
-		(property "Value" "~"
-			(at 182.5341 71.12 0)
-			(effects
-				(font
-					(size 1.27 1.27)
-				)
-				(justify left)
-			)
-		)
-		(property "Footprint" "Package_SO:SOP-8_3.9x4.9mm_P1.27mm"
-			(at 210.82 68.58 0)
-			(effects
-				(font
-					(size 1.27 1.27)
-				)
-				(hide yes)
-			)
-		)
-		(property "Datasheet" ""
-			(at 210.82 68.58 0)
-			(effects
-				(font
-					(size 1.27 1.27)
-				)
-				(hide yes)
-			)
-		)
-		(property "Description" ""
-			(at 210.82 68.58 0)
-			(effects
-				(font
-					(size 1.27 1.27)
-				)
-				(hide yes)
-			)
-		)
-		(pin "6"
-		)
-		(pin "7"
-		)
-		(pin "4"
-		)
-		(pin "5"
-		)
-		(pin "2"
-		)
-		(pin "1"
-		)
-		(pin "3"
-		)
-		(instances
-			(project "Touch Switch"
-				(path "/32e3d4f4-0c9d-4cf7-a05b-4c70ee776977"
-					(reference "S7133S1")
-					(unit 1)
-				)
-			)
-		)
-	)
-	(symbol
 		(lib_id "Relay:Relay_SPST-NO")
 		(at 55.88 134.62 0)
@@
 			)
 		)
-		(property "Footprint" "footprint:B32524R6225J000"
+		(property "Footprint" "footprint:PFR5101J400J11L4BULK"
 			(at 117.8052 31.75 0)
 			(effects
@@
 	(symbol
 		(lib_id "power:GND")
-		(at 180.34 100.33 0)
+		(at 176.53 99.06 0)
 		(unit 1)
 		(exclude_from_sim no)
@@
 		(dnp no)
 		(property "Reference" "#PWR011"
-			(at 180.34 106.68 0)
+			(at 176.53 105.41 0)
 			(effects
 				(font
@@
 		)
 		(property "Value" "GND"
-			(at 176.276 100.33 0)
+			(at 172.466 99.06 0)
 			(effects
 				(font
@@
 		)
 		(property "Footprint" ""
-			(at 180.34 100.33 0)
+			(at 176.53 99.06 0)
 			(effects
 				(font
@@
 		)
 		(property "Datasheet" ""
-			(at 180.34 100.33 0)
+			(at 176.53 99.06 0)
 			(effects
 				(font
@@
 		)
 		(property "Description" "Power symbol creates a global label with name \"GND\" , ground"
-			(at 180.34 100.33 0)
+			(at 176.53 99.06 0)
 			(effects
 				(font
@@
 			)
 		)
-		(property "Footprint" ""
+		(property "Footprint" "Connector_PinHeader_2.54mm:PinHeader_1x01_P2.54mm_Vertical"
 			(at 219.71 116.84 0)
 			(effects
@@
 			)
 		)
-		(property "Footprint" ""
+		(property "Footprint" "Connector_PinHeader_2.54mm:PinHeader_1x03_P2.54mm_Vertical"
 			(at 19.05 30.48 0)
 			(effects
@@
 			)
 		)
-		(property "Footprint" ""
+		(property "Footprint" "Connector_PinHeader_2.54mm:PinHeader_1x01_P2.54mm_Vertical"
 			(at 219.71 125.73 0)
 			(effects
@@
 			)
 		)
-		(property "Footprint" ""
+		(property "Footprint" "Connector_PinHeader_2.54mm:PinHeader_1x01_P2.54mm_Vertical"
 			(at 240.03 116.84 0)
 			(effects
@@
 	)
 	(symbol
+		(lib_name "S7133S_1")
+		(lib_id "Library:S7133S")
+		(at 180.34 83.82 0)
+		(unit 1)
+		(exclude_from_sim no)
+		(in_bom yes)
+		(on_board yes)
+		(dnp no)
+		(fields_autoplaced yes)
+		(property "Reference" "S713XS1"
+			(at 182.5341 68.58 0)
+			(effects
+				(font
+					(size 1.27 1.27)
+				)
+				(justify left)
+			)
+		)
+		(property "Value" "~"
+			(at 182.5341 71.12 0)
+			(effects
+				(font
+					(size 1.27 1.27)
+				)
+				(justify left)
+			)
+		)
+		(property "Footprint" "Package_SO:SOP-8_3.9x4.9mm_P1.27mm"
+			(at 210.82 68.58 0)
+			(effects
+				(font
+					(size 1.27 1.27)
+				)
+				(hide yes)
+			)
+		)
+		(property "Datasheet" ""
+			(at 210.82 68.58 0)
+			(effects
+				(font
+					(size 1.27 1.27)
+				)
+				(hide yes)
+			)
+		)
+		(property "Description" ""
+			(at 210.82 68.58 0)
+			(effects
+				(font
+					(size 1.27 1.27)
+				)
+				(hide yes)
+			)
+		)
+		(pin "4"
+		)
+		(pin "8"
+		)
+		(pin "6"
+		)
+		(pin "5"
+		)
+		(pin "1"
+		)
+		(pin "2"
+		)
+		(pin "7"
+		)
+		(pin "3"
+		)
+		(instances
+			(project "Touch Switch"
+				(path "/32e3d4f4-0c9d-4cf7-a05b-4c70ee776977"
+					(reference "S713XS1")
+					(unit 1)
+				)
+			)
+		)
+	)
+	(symbol
 		(lib_id "Relay:Relay_SPST-NO")
 		(at 115.57 78.74 0)
@@
 			)
 		)
-		(property "Footprint" ""
+		(property "Footprint" "Connector_PinHeader_2.54mm:PinHeader_1x01_P2.54mm_Vertical"
 			(at 240.03 125.73 0)
 			(effects
@@
 			)
 		)
-		(property "Footprint" ""
+		(property "Footprint" "footprint:transformer"
 			(at 157.48 35.56 0)
 			(effects

Commit message: PCB V2
Parts:
- R5, R6: footprint Resistor_SMD:R_1206_3216Metric -> Resistor_SMD:R_0805_2012Metric
Changed lines of the file:
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@@
 			)
 		)
-		(property "Footprint" "Resistor_SMD:R_1206_3216Metric"
+		(property "Footprint" "Resistor_SMD:R_0805_2012Metric"
 			(at 201.422 87.63 90)
 			(effects
@@
 			)
 		)
-		(property "Footprint" "Resistor_SMD:R_1206_3216Metric"
+		(property "Footprint" "Resistor_SMD:R_0805_2012Metric"
 			(at 201.422 71.12 90)
 			(effects

Commit message: End 20-05-2024
Parts:
- added H1, H2, H3, H4: MountingHole, MountingHole:MountingHole_2.2mm_M2_Pad_Via, symbol Mechanical:MountingHole

Commit message: Secondary without GND PLANE
Parts:
- removed J1: Conn_01x03_Pin, Connector_PinHeader_2.54mm:PinHeader_1x03_P2.54mm_Vertical, symbol Connector:Conn_01x03_Pin
- added J1, J7, J8: Conn_01x01_Pin, footprint:power_connector, symbol Connector:Conn_01x01_Pin
- J3, J4, J5, J6: footprint Connector_PinHeader_2.54mm:PinHeader_1x01_P2.54mm_Vertical -> footprint:power_connector
Connections:
- net L1 is gone; now on net L: F1.1
- net L: now also J1.1 (Pin_1)
- net N: now also J7.1 (Pin_1), J8.1 (Pin_1)
Changed lines of the file:
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@@
 		)
 	)
-	(global_label "L1"
+	(global_label "L"
 		(shape input)
 		(at 30.48 21.59 180)
@@
 		)
 		(property "Intersheetrefs" "${INTERSHEET_REFS}"
-			(at 25.2572 21.59 0)
+			(at 26.4667 21.59 0)
 			(effects
 				(font
@@
 	)
 	(symbol
+		(lib_id "Connector:Conn_01x01_Pin")
+		(at 19.05 27.94 0)
+		(unit 1)
+		(exclude_from_sim no)
+		(in_bom yes)
+		(on_board yes)
+		(dnp no)
+		(property "Reference" "J1"
+			(at 17.526 27.94 0)
+			(effects
+				(font
+					(size 1.27 1.27)
+				)
+			)
+		)
+		(property "Value" "Conn_01x01_Pin"
+			(at 19.685 25.4 0)
+			(effects
+				(font
+					(size 1.27 1.27)
+				)
+				(hide yes)
+			)
+		)
+		(property "Footprint" "footprint:power_connector"
+			(at 19.05 27.94 0)
+			(effects
+				(font
+					(size 1.27 1.27)
+				)
+				(hide yes)
+			)
+		)
+		(property "Datasheet" "~"
+			(at 19.05 27.94 0)
+			(effects
+				(font
+					(size 1.27 1.27)
+				)
+				(hide yes)
+			)
+		)
+		(property "Description" "Generic connector, single row, 01x01, script generated"
+			(at 19.05 27.94 0)
+			(effects
+				(font
+					(size 1.27 1.27)
+				)
+				(hide yes)
+			)
+		)
+		(pin "1"
+		)
+		(instances
+			(project "Touch Switch"
+				(path "/32e3d4f4-0c9d-4cf7-a05b-4c70ee776977"
+					(reference "J1")
+					(unit 1)
+				)
+			)
+		)
+	)
+	(symbol
 		(lib_id "Device:R")
 		(at 109.22 27.94 0)
@@
 			)
 		)
-		(property "Footprint" "Connector_PinHeader_2.54mm:PinHeader_1x01_P2.54mm_Vertical"
+		(property "Footprint" "footprint:power_connector"
 			(at 219.71 116.84 0)
 			(effects
@@
 	)
 	(symbol
-		(lib_id "Connector:Conn_01x03_Pin")
-		(at 19.05 30.48 0)
-		(unit 1)
-		(exclude_from_sim no)
-		(in_bom yes)
-		(on_board yes)
-		(dnp no)
-		(property "Reference" "J1"
-			(at 19.685 22.86 0)
-			(effects
-				(font
-					(size 1.27 1.27)
-				)
-			)
-		)
-		(property "Value" "Conn_01x03_Pin"
-			(at 19.685 25.4 0)
-			(effects
-				(font
-					(size 1.27 1.27)
-				)
-				(hide yes)
-			)
-		)
-		(property "Footprint" "Connector_PinHeader_2.54mm:PinHeader_1x03_P2.54mm_Vertical"
-			(at 19.05 30.48 0)
-			(effects
-				(font
-					(size 1.27 1.27)
-				)
-				(hide yes)
-			)
-		)
-		(property "Datasheet" "~"
-			(at 19.05 30.48 0)
-			(effects
-				(font
-					(size 1.27 1.27)
-				)
-				(hide yes)
-			)
-		)
-		(property "Description" "Generic connector, single row, 01x03, script generated"
-			(at 19.05 30.48 0)
-			(effects
-				(font
-					(size 1.27 1.27)
-				)
-				(hide yes)
-			)
-		)
-		(pin "3"
-		)
-		(pin "2"
-		)
-		(pin "1"
-		)
-		(instances
-			(project "Touch Switch"
-				(path "/32e3d4f4-0c9d-4cf7-a05b-4c70ee776977"
-					(reference "J1")
-					(unit 1)
-				)
-			)
-		)
-	)
-	(symbol
 		(lib_id "Relay:Relay_SPST-NO")
 		(at 111.76 134.62 0)
@@
 			)
 		)
-		(property "Footprint" "Connector_PinHeader_2.54mm:PinHeader_1x01_P2.54mm_Vertical"
+		(property "Footprint" "footprint:power_connector"
 			(at 219.71 125.73 0)
 			(effects
@@
 	)
 	(symbol
+		(lib_id "Connector:Conn_01x01_Pin")
+		(at 19.05 33.02 0)
+		(unit 1)
+		(exclude_from_sim no)
+		(in_bom yes)
+		(on_board yes)
+		(dnp no)
+		(property "Reference" "J8"
+			(at 17.526 33.274 0)
+			(effects
+				(font
+					(size 1.27 1.27)
+				)
+			)
+		)
+		(property "Value" "Conn_01x01_Pin"
+			(at 19.685 30.48 0)
+			(effects
+				(font
+					(size 1.27 1.27)
+				)
+				(hide yes)
+			)
+		)
+		(property "Footprint" "footprint:power_connector"
+			(at 19.05 33.02 0)
+			(effects
+				(font
+					(size 1.27 1.27)
+				)
+				(hide yes)
+			)
+		)
+		(property "Datasheet" "~"
+			(at 19.05 33.02 0)
+			(effects
+				(font
+					(size 1.27 1.27)
+				)
+				(hide yes)
+			)
+		)
+		(property "Description" "Generic connector, single row, 01x01, script generated"
+			(at 19.05 33.02 0)
+			(effects
+				(font
+					(size 1.27 1.27)
+				)
+				(hide yes)
+			)
+		)
+		(pin "1"
+		)
+		(instances
+			(project "Touch Switch"
+				(path "/32e3d4f4-0c9d-4cf7-a05b-4c70ee776977"
+					(reference "J8")
+					(unit 1)
+				)
+			)
+		)
+	)
+	(symbol
 		(lib_id "power:+3.3V")
 		(at 237.49 29.21 0)
@@
 			)
 		)
-		(property "Footprint" "Connector_PinHeader_2.54mm:PinHeader_1x01_P2.54mm_Vertical"
+		(property "Footprint" "footprint:power_connector"
 			(at 240.03 116.84 0)
 			(effects
@@
 	)
 	(symbol
+		(lib_id "Connector:Conn_01x01_Pin")
+		(at 19.05 30.48 0)
+		(unit 1)
+		(exclude_from_sim no)
+		(in_bom yes)
+		(on_board yes)
+		(dnp no)
+		(property "Reference" "J7"
+			(at 17.526 30.48 0)
+			(effects
+				(font
+					(size 1.27 1.27)
+				)
+			)
+		)
+		(property "Value" "Conn_01x01_Pin"
+			(at 19.685 27.94 0)
+			(effects
+				(font
+					(size 1.27 1.27)
+				)
+				(hide yes)
+			)
+		)
+		(property "Footprint" "footprint:power_connector"
+			(at 19.05 30.48 0)
+			(effects
+				(font
+					(size 1.27 1.27)
+				)
+				(hide yes)
+			)
+		)
+		(property "Datasheet" "~"
+			(at 19.05 30.48 0)
+			(effects
+				(font
+					(size 1.27 1.27)
+				)
+				(hide yes)
+			)
+		)
+		(property "Description" "Generic connector, single row, 01x01, script generated"
+			(at 19.05 30.48 0)
+			(effects
+				(font
+					(size 1.27 1.27)
+				)
+				(hide yes)
+			)
+		)
+		(pin "1"
+		)
+		(instances
+			(project "Touch Switch"
+				(path "/32e3d4f4-0c9d-4cf7-a05b-4c70ee776977"
+					(reference "J7")
+					(unit 1)
+				)
+			)
+		)
+	)
+	(symbol
 		(lib_id "Device:R")
 		(at 109.22 39.37 0)
@@
 			)
 		)
-		(property "Footprint" "Connector_PinHeader_2.54mm:PinHeader_1x01_P2.54mm_Vertical"
+		(property "Footprint" "footprint:power_connector"
 			(at 240.03 125.73 0)
 			(effects

Commit message: PCB V2
Parts:
- removed D1: D_Bridge_+-AA, Diode_SMD:Diode_Bridge_Diotec_ABS, symbol Device:D_Bridge_+-AA
- removed H1, H2, H3, H4: MountingHole, MountingHole:MountingHole_2.2mm_M2_Pad_Via, symbol Mechanical:MountingHole
- added D9: DF08M, Diode_SMD:Diode_Bridge_Diotec_ABS, symbol Diode_Bridge:DF08M
- C5: footprint footprint:PFR5101J400J11L4BULK -> Capacitor_SMD:C_1206_3216Metric
Connections:
- net CT1: now also Q2.1 (B), R13.1; no longer Q3.1 (B), R14.1
- net CT3: now also Q1.1 (B), R12.1; no longer Q2.1 (B), R13.1
- net CT4: now also Q3.1 (B), R14.1; no longer Q1.1 (B), R12.1
- net GND: now also D9.2 (-)
- net N: now also D9.3
- net at L1.1, R1.2: now also D9.1 (+)
- net at C7.1, F1.2: now also D9.4

Commit message: PCB V3
Other:
- moved on the sheet: C1, C2, C3, C4, C5, C6, C7, D2, D3, D4, D5, D6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
