File: control_card/control_card.kicad_pcb (KiCad board)
At the start: 2 copper layers, 72.9 x 46.5 mm, 47 parts, among them IC1 TLSR8253F512ET48, J1 Conn_02x04_Counter_Clockwise, J2 Conn_01x01_Pin, J3 Conn_01x01_Pin, J4 Conn_01x01_Pin, J5 Conn_01x01_Pin, U1 Wifi, Y1 Crystal_GND24_Small

Commit message: PCB (control_card) : modified
Parts:
- C20: moved to B.Cu
- moved L2 9.79 mm to (153.4, 75.3), turned to 0 degrees
- moved C14 6.66 mm to (154.8, 72.3), turned to 90 degrees
- moved C16 6.18 mm to (153.2, 71.9), turned to 90 degrees
- moved C15 6.17 mm to (152.5, 74.1), turned to 180 degrees
- moved AE1 5.37 mm to (156.2, 61.8)
- moved C19 4.81 mm to (152.4, 64.9), turned to 180 degrees
- moved G*** 3.66 mm to (171.5, 60.2)
- moved C18 2.98 mm to (152.4, 66.4), turned to 180 degrees
- moved L3 2.08 mm to (153.2, 68.1), turned to 90 degrees
- moved C8 1.88 mm to (153.6, 71.2)
- moved C7 1.88 mm to (152.1, 71.2)
- moved IC1 1.64 mm to (158.5, 78.0)
- moved C17 1.51 mm to (152.4, 69.7), turned to 180 degrees
- moved C20 1.45 mm to (155.9, 69.3)
- moved C3 1.31 mm to (164.3, 81.0), turned to 0 degrees
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Routing:
- net ANT: track 19.4 -> 5.45 mm
- net VANT: track 15.5 -> 3.85 mm
- net +1V2: track 33.5 -> 39.5 mm
- net RST: track 1.41 -> 5.45 mm, vias 0 -> 2
- net Net-(AE1-A): track 5.69 -> 2.47 mm
- net GND: track 29.5 -> 26.8 mm, vias 15 -> 420
- net Clock1: track 13.4 -> 15.8 mm, vias 4 -> 0
- net In_4: track 36.0 -> 38.1 mm
- net In_2: track 39.9 -> 41.7 mm
- net In_3: track 37.5 -> 39.2 mm
- net In_1: track 43.3 -> 44.9 mm
- net Sig_4: track 25.6 -> 24.5 mm
- net Sig_3: track 26.7 -> 25.7 mm
- net Net-(IC1-VDCDC_SW): track 5.55 -> 6.51 mm
- net Net-(IC1-VDCDC): track 4.60 -> 5.39 mm
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Other:
- outline, holes or cut-outs redrawn

Commit message: PCB (control_card) : Test point added
Parts:
- added SWM: TestPoint, TestPoint:TestPoint_Pad_D1.0mm, F.Cu at (153.3, 79.5)
- added SWS: TestPoint, TestPoint:TestPoint_Pad_D1.0mm, F.Cu at (161.5, 84.7)
- moved C15 0.14 mm to (152.3, 74.1)
- moved C16 0.13 mm to (153.1, 71.9)
Connections:
- IC1 pad 46: unconnected-(IC1-PD4-Pad46) -> SWM
- IC1 pad 7: unconnected-(IC1-PA5-Pad7) -> Sig_2
- IC1 pad 8: Sig_2 -> Sig_1
- IC1 pad 9: Sig_1 -> SWS
Routing:
- net SWS: track 0.00 -> 4.72 mm
- net SWM: track 0.00 -> 1.86 mm
- net Sig_1: track 29.1 -> 28.3 mm
- net Sig_2: track 30.0 -> 29.4 mm
- net GND: vias 420 -> 418
