File: control_card/control_card.kicad_pcb (KiCad board)
At the start: 2 copper layers, 72.9 x 46.5 mm, 49 parts, among them IC1 TLSR8253F512ET48, J1 Conn_02x04_Counter_Clockwise, J2 Conn_01x01_Pin, J3 Conn_01x01_Pin, J4 Conn_01x01_Pin, J5 Conn_01x01_Pin, U1 Wifi, Y1 Crystal_GND24_Small

Commit message: PCB (control_card): modified
Parts:
- moved SWS 1.84 mm to (159.7, 84.1)
Routing:
- net SWS: track 4.72 -> 2.65 mm
- net GND: vias 418 -> 423
Changed lines of the file:
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@@
 	(footprint "TestPoint:TestPoint_Pad_D1.0mm"
 		(layer "F.Cu")
-		(at 161.459339 84.660661)
+		(at 159.719339 84.060661)
 		(descr "SMD pad as test Point, diameter 1.0mm")
 		(tags "test point SMD pad")
 		(property "Reference" "SWS"
-			(at -0.03 1.49 0)
+			(at 2.43 0.01 0)
 			(layer "F.SilkS")
 			(effects
@@
 	)
 	(via
+		(at 190.726196 73.630665)
+		(size 0.6)
+		(drill 0.3)
+		(layers "F.Cu" "B.Cu")
+		(free yes)
+		(net 1)
+	)
+	(via
 		(at 170.079339 100.270661)
 		(size 0.6)
@@
 	)
 	(via
+		(at 190.728945 73.010641)
+		(size 0.6)
+		(drill 0.3)
+		(layers "F.Cu" "B.Cu")
+		(free yes)
+		(net 1)
+	)
+	(via
 		(at 134.329339 100.230661)
 		(size 0.6)
@@
 	)
 	(via
+		(at 190.726196 69.280665)
+		(size 0.6)
+		(drill 0.3)
+		(layers "F.Cu" "B.Cu")
+		(free yes)
+		(net 1)
+	)
+	(via
 		(at 184.819339 69.700661)
 		(size 0.6)
@@
 	)
 	(via
-		(at 190.679339 74.440661)
+		(at 190.722088 74.870637)
 		(size 0.6)
 		(drill 0.3)
@@
 	)
 	(via
-		(at 190.669339 71.030661)
-		(size 0.6)
-		(drill 0.3)
-		(layers "F.Cu" "B.Cu")
-		(free yes)
-		(net 1)
-	)
-	(via
 		(at 126.009339 84.120661)
 		(size 0.6)
@@
 	)
 	(via
+		(at 190.726196 71.770665)
+		(size 0.6)
+		(drill 0.3)
+		(layers "F.Cu" "B.Cu")
+		(free yes)
+		(net 1)
+	)
+	(via
 		(at 144.489339 100.260661)
 		(size 0.6)
@@
 	)
 	(via
-		(at 190.649339 68.840661)
+		(at 173.439339 100.220661)
 		(size 0.6)
 		(drill 0.3)
@@
 	)
 	(via
-		(at 173.439339 100.220661)
+		(at 126.009339 82.780661)
 		(size 0.6)
 		(drill 0.3)
@@
 	)
 	(via
-		(at 126.009339 82.780661)
+		(at 172.769339 100.230661)
 		(size 0.6)
 		(drill 0.3)
@@
 	)
 	(via
-		(at 172.769339 100.230661)
+		(at 176.129339 100.230661)
 		(size 0.6)
 		(drill 0.3)
@@
 	)
 	(via
-		(at 176.129339 100.230661)
+		(at 190.726196 71.140665)
 		(size 0.6)
 		(drill 0.3)
@@
 	)
 	(via
-		(at 190.679339 70.010661)
-		(size 0.6)
-		(drill 0.3)
-		(layers "F.Cu" "B.Cu")
-		(free yes)
-		(net 1)
-	)
-	(via
 		(at 143.209339 77.900661)
 		(size 0.6)
@@
 	)
 	(via
-		(at 190.679339 75.460661)
+		(at 190.721694 75.490617)
 		(size 0.6)
 		(drill 0.3)
@@
 	)
 	(via
-		(at 190.629339 72.740661)
-		(size 0.6)
-		(drill 0.3)
-		(layers "F.Cu" "B.Cu")
-		(free yes)
-		(net 1)
-	)
-	(via
 		(at 193.599339 100.250661)
 		(size 0.6)
@@
 	)
 	(via
+		(at 190.716196 68.600665)
+		(size 0.6)
+		(drill 0.3)
+		(layers "F.Cu" "B.Cu")
+		(free yes)
+		(net 1)
+	)
+	(via
 		(at 194.029339 61.680661)
 		(size 0.6)
@@
 	)
 	(via
+		(at 190.728945 70.520641)
+		(size 0.6)
+		(drill 0.3)
+		(layers "F.Cu" "B.Cu")
+		(free yes)
+		(net 1)
+	)
+	(via
 		(at 132.019339 81.010661)
 		(size 0.6)
@@
 	)
 	(via
-		(at 190.669339 73.600661)
+		(at 190.718945 74.250641)
 		(size 0.6)
 		(drill 0.3)
@@
 	)
 	(via
+		(at 190.729339 69.900661)
+		(size 0.6)
+		(drill 0.3)
+		(layers "F.Cu" "B.Cu")
+		(free yes)
+		(net 1)
+	)
+	(via
 		(at 144.639339 64.490661)
 		(size 0.6)
@@
 	)
 	(via
+		(at 190.729339 72.390661)
+		(size 0.6)
+		(drill 0.3)
+		(layers "F.Cu" "B.Cu")
+		(free yes)
+		(net 1)
+	)
+	(via
 		(at 189.869339 57.500661)
 		(size 0.6)
@@
 	)
 	(via
-		(at 190.619339 71.930661)
+		(at 144.289339 82.510661)
 		(size 0.6)
 		(drill 0.3)
@@
 	)
 	(via
-		(at 144.289339 82.510661)
+		(at 194.269339 100.260661)
 		(size 0.6)
 		(drill 0.3)
@@
 	)
 	(via
-		(at 194.269339 100.260661)
+		(at 190.718945 67.980641)
 		(size 0.6)
 		(drill 0.3)
@@
 	)
 	(segment
-		(start 165.639339 76.030661)
-		(end 165.854339 76.030661)
-		(width 0.2)
-		(layer "F.Cu")
-		(net 4)
-	)
-	(segment
 		(start 164.949339 76.040661)
 		(end 165.249339 76.040661)
@@
 	)
 	(segment
-		(start 165.854339 76.030661)
-		(end 166.759339 75.125661)
+		(start 154.346973 76.390661)
+		(end 152.409339 76.390661)
 		(width 0.2)
 		(layer "F.Cu")
@@
 	)
 	(segment
-		(start 154.346973 76.390661)
-		(end 152.409339 76.390661)
+		(start 163.864411 76.820661)
+		(end 164.809339 76.820661)
 		(width 0.2)
 		(layer "F.Cu")
@@
 	)
 	(segment
-		(start 163.864411 76.820661)
-		(end 164.809339 76.820661)
+		(start 166.379339 76.030661)
+		(end 166.759339 75.650661)
 		(width 0.2)
 		(layer "F.Cu")
@@
 	)
 	(segment
+		(start 166.759339 75.650661)
+		(end 166.759339 75.125661)
+		(width 0.2)
+		(layer "F.Cu")
+		(net 4)
+	)
+	(segment
 		(start 164.949339 76.040661)
 		(end 165.029339 75.960661)
@@
 	)
 	(segment
+		(start 165.639339 76.030661)
+		(end 166.379339 76.030661)
+		(width 0.2)
+		(layer "F.Cu")
+		(net 4)
+	)
+	(segment
 		(start 165.249339 76.040661)
 		(end 165.179339 75.970661)
@@
 	)
 	(segment
-		(start 160.099339 84.660661)
-		(end 161.459339 84.660661)
-		(width 0.2)
-		(layer "F.Cu")
-		(net 38)
-	)
-	(segment
-		(start 159.709339 84.270661)
-		(end 160.099339 84.660661)
+		(start 159.709339 84.020661)
+		(end 159.769339 84.080661)
 		(width 0.2)
 		(layer "F.Cu")
@@
 	(segment
 		(start 159.709339 81.458161)
-		(end 159.709339 84.270661)
+		(end 159.709339 84.020661)
 		(width 0.2)
 		(layer "F.Cu")
@@
 	)
 	(segment
-		(start 157.199339 70.080661)
-		(end 157.199339 74.573161)
+		(start 159.049339 68.610661)
+		(end 157.199339 70.460661)
 		(width 0.2)
 		(layer "F.Cu")
@@
 	)
 	(segment
-		(start 188.805001 65.954999)
-		(end 188.805001 64.600001)
+		(start 157.199339 74.573161)
+		(end 157.209339 74.583161)
 		(width 0.2)
 		(layer "F.Cu")
@@
 	)
 	(segment
-		(start 159.049339 68.210001)
-		(end 159.049999 68.210661)
+		(start 188.805001 65.954999)
+		(end 188.805001 64.600001)
 		(width 0.2)
 		(layer "F.Cu")
@@
 	)
 	(segment
-		(start 159.049339 68.610661)
-		(end 158.114339 69.545661)
+		(start 159.049339 68.210001)
+		(end 159.049999 68.210661)
 		(width 0.2)
 		(layer "F.Cu")
@@
 	)
 	(segment
-		(start 157.199339 74.573161)
-		(end 157.209339 74.583161)
-		(width 0.2)
-		(layer "F.Cu")
-		(net 50)
-	)
-	(segment
 		(start 188.529339 66.160661)
 		(end 188.549339 66.140661)
@@
 	)
 	(segment
-		(start 157.734339 69.545661)
-		(end 157.199339 70.080661)
-		(width 0.2)
-		(layer "F.Cu")
-		(net 50)
-	)
-	(segment
-		(start 158.114339 69.545661)
-		(end 157.734339 69.545661)
+		(start 157.199339 70.460661)
+		(end 157.199339 74.573161)
 		(width 0.2)
 		(layer "F.Cu")
@@
 	)
 	(segment
+		(start 153.929339 79.500661)
+		(end 154.199339 79.770661)
+		(width 0.2)
+		(layer "F.Cu")
+		(net 74)
+	)
+	(segment
 		(start 153.269339 79.500661)
-		(end 153.539339 79.770661)
+		(end 153.929339 79.500661)
 		(width 0.2)
 		(layer "F.Cu")
@@
 	)
 	(segment
-		(start 153.539339 79.770661)
+		(start 154.199339 79.770661)
 		(end 155.021839 79.770661)
 		(width 0.2)
